Commit message: Update joints & links' name

File: Spot-Arm/spot_arm_description/urdf/spot_arm.xacro (robot description, xacro)
@@ -24,5 +24,5 @@
   </collision>
 </link>
-<link name="Part3_1">
+<link name="link4">
   <inertial>
     <origin rpy="0 0 0" xyz="-0.00911464892336129 0.12606054498393937 5.551115123125783e-17"/>
@@ -33,5 +33,5 @@
     <origin rpy="0 0 0" xyz="0.001 -0.4505 -0.0475"/>
     <geometry>
-      <mesh filename="package://spot_arm_description/meshes/Part3_1.stl" scale="0.001 0.001 0.001"/>
+      <mesh filename="package://spot_arm_description/meshes/link4.stl" scale="0.001 0.001 0.001"/>
     </geometry>
     <material name="silver"/>
@@ -40,9 +40,9 @@
     <origin rpy="0 0 0" xyz="0.001 -0.4505 -0.0475"/>
     <geometry>
-      <mesh filename="package://spot_arm_description/meshes/Part3_1.stl" scale="0.001 0.001 0.001"/>
-    </geometry>
-  </collision>
-</link>
-<link name="gripper_1">
+      <mesh filename="package://spot_arm_description/meshes/link4.stl" scale="0.001 0.001 0.001"/>
+    </geometry>
+  </collision>
+</link>
+<link name="gripper">
   <inertial>
     <origin rpy="0 0 0" xyz="-8.366123908053191e-08 0.07051371901138614 0.017123167388316526"/>
@@ -53,5 +53,5 @@
     <origin rpy="0 0 0" xyz="0.0085 -0.77959 -0.0475"/>
     <geometry>
-      <mesh filename="package://spot_arm_description/meshes/gripper_1.stl" scale="0.001 0.001 0.001"/>
+      <mesh filename="package://spot_arm_description/meshes/gripper.stl" scale="0.001 0.001 0.001"/>
     </geometry>
     <material name="silver"/>
@@ -60,9 +60,9 @@
     <origin rpy="0 0 0" xyz="0.0085 -0.77959 -0.0475"/>
     <geometry>
-      <mesh filename="package://spot_arm_description/meshes/gripper_1.stl" scale="0.001 0.001 0.001"/>
-    </geometry>
-  </collision>
-</link>
-<link name="finger_1">
+      <mesh filename="package://spot_arm_description/meshes/gripper.stl" scale="0.001 0.001 0.001"/>
+    </geometry>
+  </collision>
+</link>
+<link name="finger">
   <inertial>
     <origin rpy="0 0 0" xyz="0.8635899028063472 0.09862056591557622 0.00850232975194119"/>
@@ -73,5 +73,5 @@
     <origin rpy="0 0 0" xyz="0.87709 -0.823505 -0.0185"/>
     <geometry>
-      <mesh filename="package://spot_arm_description/meshes/finger_1.stl" scale="0.001 0.001 0.001"/>
+      <mesh filename="package://spot_arm_description/meshes/finger.stl" scale="0.001 0.001 0.001"/>
     </geometry>
     <material name="silver"/>
@@ -80,9 +80,9 @@
     <origin rpy="0 0 0" xyz="0.87709 -0.823505 -0.0185"/>
     <geometry>
-      <mesh filename="package://spot_arm_description/meshes/finger_1.stl" scale="0.001 0.001 0.001"/>
-    </geometry>
-  </collision>
-</link>
-<link name="Part1_1">
+      <mesh filename="package://spot_arm_description/meshes/finger.stl" scale="0.001 0.001 0.001"/>
+    </geometry>
+  </collision>
+</link>
+<link name="link2">
   <inertial>
     <origin rpy="0 0 0" xyz="-0.0163095589512068 0.17540914221218962 0.0"/>
@@ -93,5 +93,5 @@
     <origin rpy="0 0 0" xyz="-0.015 -0.0 -0.115"/>
     <geometry>
-      <mesh filename="package://spot_arm_description/meshes/Part1_1.stl" scale="0.001 0.001 0.001"/>
+      <mesh filename="package://spot_arm_description/meshes/link2.stl" scale="0.001 0.001 0.001"/>
     </geometry>
     <material name="silver"/>
@@ -100,9 +100,9 @@
     <origin rpy="0 0 0" xyz="-0.015 -0.0 -0.115"/>
     <geometry>
-      <mesh filename="package://spot_arm_description/meshes/Part1_1.stl" scale="0.001 0.001 0.001"/>
-    </geometry>
-  </collision>
-</link>
-<link name="Part0_1">
+      <mesh filename="package://spot_arm_description/meshes/link2.stl" scale="0.001 0.001 0.001"/>
+    </geometry>
+  </collision>
+</link>
+<link name="link1">
   <inertial>
     <origin rpy="0 0 0" xyz="0.05071972800114364 -1.0308563411658574e-17 0.04676911608650795"/>
@@ -113,5 +113,5 @@
     <origin rpy="0 0 0" xyz="-0.0 -0.0 -0.065"/>
     <geometry>
-      <mesh filename="package://spot_arm_description/meshes/Part0_1.stl" scale="0.001 0.001 0.001"/>
+      <mesh filename="package://spot_arm_description/meshes/link1.stl" scale="0.001 0.001 0.001"/>
     </geometry>
     <material name="silver"/>
@@ -120,9 +120,9 @@
     <origin rpy="0 0 0" xyz="-0.0 -0.0 -0.065"/>
     <geometry>
-      <mesh filename="package://spot_arm_description/meshes/Part0_1.stl" scale="0.001 0.001 0.001"/>
-    </geometry>
-  </collision>
-</link>
-<link name="Part4_1">
+      <mesh filename="package://spot_arm_description/meshes/link1.stl" scale="0.001 0.001 0.001"/>
+    </geometry>
+  </collision>
+</link>
+<link name="wrist">
   <inertial>
     <origin rpy="0 0 0" xyz="0.03954999709763633 0.03472006124891969 4.209155544249166e-08"/>
@@ -133,5 +133,5 @@
     <origin rpy="0 0 0" xyz="0.0485 -0.69859 -0.0475"/>
     <geometry>
-      <mesh filename="package://spot_arm_description/meshes/Part4_1.stl" scale="0.001 0.001 0.001"/>
+      <mesh filename="package://spot_arm_description/meshes/wrist.stl" scale="0.001 0.001 0.001"/>
     </geometry>
     <material name="silver"/>
@@ -140,9 +140,9 @@
     <origin rpy="0 0 0" xyz="0.0485 -0.69859 -0.0475"/>
     <geometry>
-      <mesh filename="package://spot_arm_description/meshes/Part4_1.stl" scale="0.001 0.001 0.001"/>
-    </geometry>
-  </collision>
-</link>
-<link name="Part2_1">
+      <mesh filename="package://spot_arm_description/meshes/wrist.stl" scale="0.001 0.001 0.001"/>
+    </geometry>
+  </collision>
+</link>
+<link name="link3">
   <inertial>
     <origin rpy="0 0 0" xyz="-0.015621881612358529 0.06665620790957599 -0.058074231003688394"/>
@@ -153,5 +153,5 @@
     <origin rpy="0 0 0" xyz="-0.017 -0.3125 -0.115"/>
     <geometry>
-      <mesh filename="package://spot_arm_description/meshes/Part2_1.stl" scale="0.001 0.001 0.001"/>
+      <mesh filename="package://spot_arm_description/meshes/link3.stl" scale="0.001 0.001 0.001"/>
     </geometry>
     <material name="silver"/>
@@ -160,56 +160,56 @@
     <origin rpy="0 0 0" xyz="-0.017 -0.3125 -0.115"/>
     <geometry>
-      <mesh filename="package://spot_arm_description/meshes/Part2_1.stl" scale="0.001 0.001 0.001"/>
-    </geometry>
-  </collision>
-</link>
-<joint name="Rev3" type="revolute">
+      <mesh filename="package://spot_arm_description/meshes/link3.stl" scale="0.001 0.001 0.001"/>
+    </geometry>
+  </collision>
+</link>
+<joint name="Joint1" type="revolute">
+  <origin rpy="0 0 0" xyz="0.0 0.0 0.065"/>
+  <parent link="base_link"/>
+  <child link="link1"/>
+  <axis xyz="0.0 0.0 1.0"/>
+  <limit effort="100" lower="-3.141593" upper="2.617994" velocity="100"/>
+</joint>
+<joint name="Joint2" type="revolute">
+  <origin rpy="0 0 0" xyz="0.015 0.0 0.05"/>
+  <parent link="link1"/>
+  <child link="link2"/>
+  <axis xyz="-1.0 0.0 0.0"/>
+  <limit effort="100" lower="-3.665191" upper="0.0" velocity="100"/>
+</joint>
+<joint name="Joint3" type="revolute">
+  <origin rpy="0 0 0" xyz="0.002 0.3125 0.0"/>
+  <parent link="link2"/>
+  <child link="link3"/>
+  <axis xyz="1.0 0.0 0.0"/>
+  <limit effort="100" lower="0.0" upper="2.96706" velocity="100"/>
+</joint>
+<joint name="Joint4" type="revolute">
   <origin rpy="0 0 0" xyz="-0.018 0.138 -0.0675"/>
-  <parent link="Part2_1"/>
-  <child link="Part3_1"/>
+  <parent link="link3"/>
+  <child link="link4"/>
   <axis xyz="0.0 1.0 0.0"/>
   <limit effort="100" lower="-2.879793" upper="2.879793" velocity="100"/>
 </joint>
-<joint name="Rev6" type="revolute">
+<joint name="Joint5" type="revolute">
+  <origin rpy="0 0 0" xyz="-0.0475 0.24809 0.0"/>
+  <parent link="link4"/>
+  <child link="wrist"/>
+  <axis xyz="1.0 0.0 0.0"/>
+  <limit effort="100" lower="-1.570796" upper="1.570796" velocity="100"/>
+</joint>
+<joint name="Joint6" type="revolute">
   <origin rpy="0 0 0" xyz="0.04 0.081 0.0"/>
-  <parent link="Part4_1"/>
-  <child link="gripper_1"/>
+  <parent link="wrist"/>
+  <child link="gripper"/>
   <axis xyz="-0.0 1.0 0.0"/>
   <limit effort="100" lower="-2.96706" upper="2.96706" velocity="100"/>
 </joint>
-<joint name="Rev7" type="revolute">
+<joint name="Joint7" type="revolute">
   <origin rpy="0 0 0" xyz="-0.86859 0.043915 -0.029"/>
-  <parent link="gripper_1"/>
-  <child link="finger_1"/>
+  <parent link="gripper"/>
+  <child link="finger"/>
   <axis xyz="1.0 -0.0 0.0"/>
   <limit effort="100" lower="-1.396263" upper="0.349066" velocity="100"/>
 </joint>
-<joint name="Rev8" type="revolute">
-  <origin rpy="0 0 0" xyz="0.015 0.0 0.05"/>
-  <parent link="Part0_1"/>
-  <child link="Part1_1"/>
-  <axis xyz="-1.0 0.0 0.0"/>
-  <limit effort="100" lower="-3.665191" upper="0.0" velocity="100"/>
-</joint>
-<joint name="Rev9" type="revolute">
-  <origin rpy="0 0 0" xyz="0.0 0.0 0.065"/>
-  <parent link="base_link"/>
-  <child link="Part0_1"/>
-  <axis xyz="0.0 0.0 1.0"/>
-  <limit effort="100" lower="-3.141593" upper="2.617994" velocity="100"/>
-</joint>
-<joint name="Rev10" type="revolute">
-  <origin rpy="0 0 0" xyz="-0.0475 0.24809 0.0"/>
-  <parent link="Part3_1"/>
-  <child link="Part4_1"/>
-  <axis xyz="1.0 0.0 0.0"/>
-  <limit effort="100" lower="-1.570796" upper="1.570796" velocity="100"/>
-</joint>
-<joint name="Rev11" type="revolute">
-  <origin rpy="0 0 0" xyz="0.002 0.3125 0.0"/>
-  <parent link="Part1_1"/>
-  <child link="Part2_1"/>
-  <axis xyz="1.0 0.0 0.0"/>
-  <limit effort="100" lower="0.0" upper="2.96706" velocity="100"/>
-</joint>
 </robot>

Commit message: updated urdf to include arm

File: Spot-Arm/spot_arm_description/urdf/spot_arm.xacro (robot description, xacro)
@@ -4,5 +4,5 @@
 <xacro:include filename="$(find spot_arm_description)/urdf/spot_arm.trans" />
 <xacro:include filename="$(find spot_arm_description)/urdf/spot_arm.gazebo" />
-<link name="base_link">
+<link name="base_arm_link">
   <inertial>
     <origin rpy="0 0 0" xyz="1.2371844231029972e-17 0.0 0.0325"/>
@@ -164,7 +164,12 @@
   </collision>
 </link>
+<joint name="base_arm_joint" type="fixed">
+        <origin xyz="0.29 0 0.08" rpy="0 0 0" />
+        <parent link="body" />
+        <child link="base_arm_link" />
+    </joint>
 <joint name="Joint1" type="revolute">
   <origin rpy="0 0 0" xyz="0.0 0.0 0.065"/>
-  <parent link="base_link"/>
+  <parent link="base_arm_link"/>
   <child link="link1"/>
   <axis xyz="0.0 0.0 1.0"/>

File: spot_description/urdf/accessories.urdf.xacro (robot description, xacro)
@@ -72,3 +72,6 @@
     </xacro:if>
   </xacro:if>
+  <xacro:if value="$(optenv SPOT_ARM 0)">
+    <xacro:include filename="$(find spot_arm_description)/urdf/spot_arm.xacro" />
+  </xacro:if>
 </robot>
