Commit message: adressed layout review comments

File: spot_description/urdf/spot_arm.xacro (robot description, xacro)
@@ -169,5 +169,5 @@
         <child link="base_arm_link" />
     </joint>
-<joint name="Joint1" type="revolute">
+<joint name="arm_joint1" type="revolute">
   <origin rpy="0 0 0" xyz="0.0 0.0 0.065"/>
   <parent link="base_arm_link"/>
@@ -176,5 +176,5 @@
   <limit effort="100" lower="-3.141593" upper="2.617994" velocity="100"/>
 </joint>
-<joint name="Joint2" type="revolute">
+<joint name="arm_joint2" type="revolute">
   <origin rpy="0 0 0" xyz="0.015 0.0 0.05"/>
   <parent link="link1"/>
@@ -183,5 +183,5 @@
   <limit effort="100" lower="-3.665191" upper="0.0" velocity="100"/>
 </joint>
-<joint name="Joint3" type="revolute">
+<joint name="arm_joint3" type="revolute">
   <origin rpy="0 0 0" xyz="0.002 0.3125 0.0"/>
   <parent link="link2"/>
@@ -190,5 +190,5 @@
   <limit effort="100" lower="0.0" upper="2.96706" velocity="100"/>
 </joint>
-<joint name="Joint4" type="revolute">
+<joint name="arm_joint4" type="revolute">
   <origin rpy="0 0 0" xyz="-0.018 0.138 -0.0675"/>
   <parent link="link3"/>
@@ -197,5 +197,5 @@
   <limit effort="100" lower="-2.879793" upper="2.879793" velocity="100"/>
 </joint>
-<joint name="Joint5" type="revolute">
+<joint name="arm_joint5" type="revolute">
   <origin rpy="0 0 0" xyz="-0.0475 0.24809 0.0"/>
   <parent link="link4"/>
@@ -204,5 +204,5 @@
   <limit effort="100" lower="-1.570796" upper="1.570796" velocity="100"/>
 </joint>
-<joint name="Joint6" type="revolute">
+<joint name="arm_joint6" type="revolute">
   <origin rpy="0 0 0" xyz="0.04 0.081 0.0"/>
   <parent link="wrist"/>
@@ -211,5 +211,5 @@
   <limit effort="100" lower="-2.96706" upper="2.96706" velocity="100"/>
 </joint>
-<joint name="Joint7" type="revolute">
+<joint name="arm_gripper" type="revolute">
   <origin rpy="0 0 0" xyz="-0.86859 0.043915 -0.029"/>
   <parent link="gripper"/>

Commit message: Fixes arm xacro for hachi.

File: spot_description/urdf/spot_arm.xacro (robot description, xacro)
@@ -165,5 +165,5 @@
 </link>
 <joint name="base_arm_joint" type="fixed">
-        <origin xyz="0.29 0 0.08" rpy="0 0 0" />
+        <origin xyz="0.29 0 0.08" rpy="0 0 -1.571" />
         <parent link="body" />
         <child link="base_arm_link" />
@@ -184,5 +184,5 @@
 </joint>
 <joint name="arm_joint3" type="revolute">
-  <origin rpy="0 0 0" xyz="0.002 0.3125 0.0"/>
+  <origin rpy="0 3.1415 0" xyz="0.002 0.3125 0.0"/>
   <parent link="link2"/>
   <child link="link3"/>

Commit message: Fixes finger frame.

File: spot_description/urdf/spot_arm.xacro (robot description, xacro)
@@ -71,5 +71,5 @@
   </inertial>
   <visual>
-    <origin rpy="0 0 0" xyz="0.87709 -0.823505 -0.0185"/>
+    <origin rpy="0 0 0" xyz="0.0145 -0.823505 -0.0185"/>
     <geometry>
       <mesh filename="package://spot_description/meshes/arm/finger.stl" scale="0.001 0.001 0.001"/>
@@ -78,5 +78,5 @@
   </visual>
   <collision>
-    <origin rpy="0 0 0" xyz="0.87709 -0.823505 -0.0185"/>
+    <origin rpy="0 0 0" xyz="0.0145 -0.823505 -0.0185"/>
     <geometry>
       <mesh filename="package://spot_description/meshes/arm/finger.stl" scale="0.001 0.001 0.001"/>
@@ -212,5 +212,5 @@
 </joint>
 <joint name="arm_gripper" type="revolute">
-  <origin rpy="0 0 0" xyz="-0.86859 0.043915 -0.029"/>
+  <origin rpy="0 0 0" xyz="0.0 0.043915 -0.029"/>
   <parent link="gripper"/>
   <child link="finger"/>
