Commit message: Replace broken URDF with fixed URDF from ROS 2 driver

File: spot_description/urdf/accessories.urdf.xacro (robot description, xacro)
@@ -10,15 +10,15 @@
       <visual>
         <geometry>
-          <mesh filename="package://spot_description/meshes/pack_top.dae"/>
+          <mesh filename="package://spot_description/meshes/base/visual/pack_top.obj"/>
         </geometry>
       </visual>
       <visual>
         <geometry>
-          <mesh filename="package://spot_description/meshes/pack_body.dae"/>
+          <mesh filename="package://spot_description/meshes/base/visual/pack_body.obj"/>
         </geometry>
       </visual>
       <collision>
         <geometry>
-          <mesh filename="package://spot_description/meshes/pack_body.dae"/>
+          <mesh filename="package://spot_description/meshes/base/visual/pack_body.obj"/>
         </geometry>
       </collision>
@@ -34,10 +34,10 @@
       <visual>
         <geometry>
-          <mesh filename="package://spot_description/meshes/lidar_mount.dae"/>
+          <mesh filename="package://spot_description/meshes/base/visual/lidar_mount.obj"/>
         </geometry>
       </visual>
       <collision>
         <geometry>
-          <mesh filename="package://spot_description/meshes/lidar_mount_collision.stl"/>
+          <mesh filename="package://spot_description/meshes/base/collision/lidar_mount_collision.stl"/>
         </geometry>
       </collision>
@@ -53,5 +53,5 @@
         <visual>
           <geometry>
-            <mesh filename="package://spot_description/meshes/velodyne_cage.stl" scale="0.001 0.001 0.001" />
+            <mesh filename="package://spot_description/meshes/base/collision/velodyne_cage.stl" scale="0.001 0.001 0.001" />
           </geometry>
           <origin xyz="0 0 0" rpy="0 0 0" />
@@ -60,5 +60,5 @@
         <collision>
           <geometry>
-            <mesh filename="package://spot_description/meshes/velodyne_cage.stl" scale="0.001 0.001 0.001" />
+            <mesh filename="package://spot_description/meshes/base/collision/velodyne_cage.stl" scale="0.001 0.001 0.001" />
           </geometry>
           <origin xyz="0 0 0" rpy="0 0 0" />
@@ -72,6 +72,3 @@
     </xacro:if>
   </xacro:if>
-  <xacro:if value="$(optenv SPOT_ARM 0)">
-    <xacro:include filename="$(find spot_description)/urdf/spot_arm.xacro" />
-  </xacro:if>
 </robot>

File: spot_description/urdf/spot.urdf.xacro (robot description, xacro)
@@ -1,277 +1,13 @@
 <?xml version="1.0" ?>
 <robot name="spot" xmlns:xacro="http://www.ros.org/wiki/xacro">
-    <link name="body">
-        <visual>
-            <geometry>
-                <mesh filename="package://spot_description/meshes/body.dae" />
-            </geometry>
-        </visual>
-        <collision>
-            <geometry>
-                <mesh filename="package://spot_description/meshes/body_collision.stl" />
-            </geometry>
-        </collision>
-    </link>
-    <link name="base_link"/>
-    <joint name="base_link_joint" type="fixed">
-        <origin xyz="0 0 0" rpy="0 0 0" />
-        <parent link="body" />
-        <child link="base_link" />
-    </joint>
-    <link name="front_rail"/>
-    <joint name="front_rail_joint" type="fixed">
-        <origin xyz="0.223 0 0.0805" rpy="0 0 0" />
-        <parent link="body" />
-        <child link="front_rail" />
-    </joint>
-    <link name="real_front_rail"/>
-    <joint name="real_front_rail_joint" type="fixed">
-        <origin xyz="0.2075 0 0.0805" rpy="0 0 0" />
-        <parent link="body" />
-        <child link="real_front_rail" />
-    </joint>
-    <link name="rear_rail"/>
-    <joint name="rear_rail_joint" type="fixed">
-        <origin xyz="-0.223 0 0.0805" rpy="0 0 0" />
-        <parent link="body" />
-        <child link="rear_rail" />
-    </joint>
-    <link name="real_rear_rail"/>
-    <joint name="real_rear_rail_joint" type="fixed">
-        <origin xyz="-0.415 0 0" rpy="0 0 0" />
-        <parent link="real_front_rail" />
-        <child link="real_rear_rail" />
-    </joint>
-    <link name="front_left_hip">
-        <visual>
-            <geometry>
-                <mesh filename="package://spot_description/meshes/front_left_hip.dae" />
-            </geometry>
-        </visual>
-        <collision>
-            <geometry>
-                <mesh filename="package://spot_description/meshes/front_left_hip_collision.stl" />
-            </geometry>
-        </collision>
-    </link>
-    <joint name="front_left_hip_x" type="revolute">
-        <origin xyz="0.29785 0.05500 0.00000" rpy="0 0 0" />
-        <axis xyz="1 0 0" />
-        <parent link="body" />
-        <child link="front_left_hip" />
-        <limit effort="1000" velocity="1000.00" lower="-0.78539816339744827899" upper="0.78539816339744827899" />
-    </joint>
-    <link name="front_left_upper_leg">
-        <visual>
-            <geometry>
-                <mesh filename="package://spot_description/meshes/front_left_upper_leg.dae" />
-            </geometry>
-        </visual>
-        <collision>
-            <geometry>
-                <mesh filename="package://spot_description/meshes/front_left_upper_leg_collision.stl" />
-            </geometry>
-        </collision>
-    </link>
-    <joint name="front_left_hip_y" type="revolute">
-        <origin xyz="0.0 0.110945 0.0" rpy="0 0 0" />
-        <axis xyz="0 1 0" />
-        <parent link="front_left_hip" />
-        <child link="front_left_upper_leg" />
-        <limit effort="1000" velocity="1000.00" lower="-0.89884456477707963539" upper="2.2951079663725435509" />
-    </joint>
-    <link name="front_left_lower_leg">
-        <visual>
-            <geometry>
-                <mesh filename="package://spot_description/meshes/front_left_lower_leg.dae" />
-            </geometry>
-        </visual>
-        <collision>
-            <geometry>
-                <mesh filename="package://spot_description/meshes/front_left_lower_leg_collision.stl" />
-            </geometry>
-        </collision>
-    </link>
-    <joint name="front_left_knee" type="revolute">
-        <origin xyz="0.025 0.000 -0.3205" rpy="0 0 0" />
-        <axis xyz="0 1 0" />
-        <parent link="front_left_upper_leg" />
-        <child link="front_left_lower_leg" />
-        <limit effort="1000" velocity="1000.00" lower="-2.7929" upper="-0.254801" />
-    </joint>
-    <link name="front_right_hip">
-        <visual>
-            <geometry>
-                <mesh filename="package://spot_description/meshes/front_right_hip.dae" />
-            </geometry>
-        </visual>
-        <collision>
-            <geometry>
-                <mesh filename="package://spot_description/meshes/front_right_hip_collision.stl" />
-            </geometry>
-        </collision>
-    </link>
-    <joint name="front_right_hip_x" type="revolute">
-        <origin xyz="0.29785 -0.05500 0.00000" rpy="0 0 0" />
-        <axis xyz="1 0 0" />
-        <parent link="body" />
-        <child link="front_right_hip" />
-        <limit effort="1000" velocity="1000.00" lower="-0.78539816339744827899" upper="0.78539816339744827899" />
-    </joint>
-    <link name="front_right_upper_leg">
-        <visual>
-            <geometry>
-                <mesh filename="package://spot_description/meshes/front_right_upper_leg.dae" />
-            </geometry>
-        </visual>
-        <collision>
-            <geometry>
-                <mesh filename="package://spot_description/meshes/front_right_upper_leg_collision.stl" />
-            </geometry>
-        </collision>
-    </link>
-    <joint name="front_right_hip_y" type="revolute">
-        <origin xyz="0.0 -0.110945 0.0" rpy="0 0 0" />
-        <axis xyz="0 1 0" />
-        <parent link="front_right_hip" />
-        <child link="front_right_upper_leg" />
-        <limit effort="1000" velocity="1000.00" lower="-0.89884456477707963539" upper="2.2951079663725435509" />
-    </joint>
-    <link name="front_right_lower_leg">
-        <visual>
-            <geometry>
-                <mesh filename="package://spot_description/meshes/front_right_lower_leg.dae" />
-            </geometry>
-        </visual>
-        <collision>
-            <geometry>
-                <mesh filename="package://spot_description/meshes/front_right_lower_leg_collision.stl" />
-            </geometry>
-        </collision>
-    </link>
-    <joint name="front_right_knee" type="revolute">
-        <origin xyz="0.025 0.000 -0.3205" rpy="0 0 0" />
-        <axis xyz="0 1 0" />
-        <parent link="front_right_upper_leg" />
-        <child link="front_right_lower_leg" />
-        <limit effort="1000" velocity="1000.00" lower="-2.7929" upper="-0.247563" />
-    </joint>
-    <link name="rear_left_hip">
-        <visual>
-            <geometry>
-                <mesh filename="package://spot_description/meshes/rear_left_hip.dae" />
-            </geometry>
-        </visual>
-        <collision>
-            <geometry>
-                <mesh filename="package://spot_description/meshes/rear_left_hip_collision.stl" />
-            </geometry>
-        </collision>
-    </link>
-    <joint name="rear_left_hip_x" type="revolute">
-        <origin xyz="-0.29785 0.05500 0.00000" rpy="0 0 0" />
-        <axis xyz="1 0 0" />
-        <parent link="body" />
-        <child link="rear_left_hip" />
-        <limit effort="1000" velocity="1000.00" lower="-0.78539816339744827899" upper="0.78539816339744827899" />
-    </joint>
-    <link name="rear_left_upper_leg">
-        <visual>
-            <geometry>
-                <mesh filename="package://spot_description/meshes/rear_left_upper_leg.dae" />
-            </geometry>
-        </visual>
-        <collision>
-            <geometry>
-                <mesh filename="package://spot_description/meshes/rear_left_upper_leg_collision.stl" />
-            </geometry>
-        </collision>
-    </link>
-    <joint name="rear_left_hip_y" type="revolute">
-        <origin xyz="0.0 0.110945 0.0" rpy="0 0 0" />
-        <axis xyz="0 1 0" />
-        <parent link="rear_left_hip" />
-        <child link="rear_left_upper_leg" />
-        <limit effort="1000" velocity="1000.00" lower="-0.89884456477707963539" upper="2.2951079663725435509" />
-    </joint>
-    <link name="rear_left_lower_leg">
-        <visual>
-            <geometry>
-                <mesh filename="package://spot_description/meshes/rear_left_lower_leg.dae" />
-            </geometry>
-        </visual>
-        <collision>
-            <geometry>
-                <mesh filename="package://spot_description/meshes/rear_left_lower_leg_collision.stl" />
-            </geometry>
-        </collision>
-    </link>
-    <joint name="rear_left_knee" type="revolute">
-        <origin xyz="0.025 0.000 -0.3205" rpy="0 0 0" />
-        <axis xyz="0 1 0" />
-        <parent link="rear_left_upper_leg" />
-        <child link="rear_left_lower_leg" />
-        <limit effort="1000" velocity="1000.00" lower="-2.7929" upper="-0.267153" />
-    </joint>
-    <link name="rear_right_hip">
-        <visual>
-            <geometry>
-                <mesh filename="package://spot_description/meshes/rear_right_hip.dae" />
-            </geometry>
-        </visual>
-        <collision>
-            <geometry>
-                <mesh filename="package://spot_description/meshes/rear_right_hip_collision.stl" />
-            </geometry>
-        </collision>
-    </link>
-    <joint name="rear_right_hip_x" type="revolute">
-        <origin xyz="-0.29785 -0.05500 0.00000" rpy="0 0 0" />
-        <axis xyz="1 0 0" />
-        <parent link="body" />
-        <child link="rear_right_hip" />
-        <limit effort="1000" velocity="1000.00" lower="-0.78539816339744827899" upper="0.78539816339744827899" />
-    </joint>
-    <link name="rear_right_upper_leg">
-        <visual>
-            <geometry>
-                <mesh filename="package://spot_description/meshes/rear_right_upper_leg.dae" />
-            </geometry>
-        </visual>
-        <collision>
-            <geometry>
-                <mesh filename="package://spot_description/meshes/rear_right_upper_leg_collision.stl" />
-            </geometry>
-        </collision>
-    </link>
-    <joint name="rear_right_hip_y" type="revolute">
-        <origin xyz="0.0 -0.110945 0.0" rpy="0 0 0" />
-        <axis xyz="0 1 0" />
-        <parent link="rear_right_hip" />
-        <child link="rear_right_upper_leg" />
-        <limit effort="1000" velocity="1000.00" lower="-0.89884456477707963539" upper="2.2951079663725435509" />
-    </joint>
-    <link name="rear_right_lower_leg">
-        <visual>
-            <geometry>
-                <mesh filename="package://spot_description/meshes/rear_right_lower_leg.dae" />
-            </geometry>
-        </visual>
-        <collision>
-            <geometry>
-                <mesh filename="package://spot_description/meshes/rear_right_lower_leg_collision.stl" />
-            </geometry>
-        </collision>
-    </link>
-    <joint name="rear_right_knee" type="revolute">
-        <origin xyz="0.025 0.000 -0.3205" rpy="0 0 0" />
-        <axis xyz="0 1 0" />
-        <parent link="rear_right_upper_leg" />
-        <child link="rear_right_lower_leg" />
-        <limit effort="1000" velocity="1000.00" lower="-2.7929" upper="-0.257725" />
-    </joint>
-    <!-- Standard accessories. -->
-    <xacro:include filename="$(find spot_description)/urdf/accessories.urdf.xacro" />
-    <!-- Optional custom includes. -->
-    <xacro:include filename="$(optenv SPOT_URDF_EXTRAS empty.urdf)" />
+  <xacro:include filename="$(find spot_description)/urdf/spot_macro.xacro" />
+  <!-- Parameters -->
+  <xacro:arg name="arm" default="false" />
+  <xacro:arg name="feet" default="false" />
+  <xacro:arg name="tf_prefix" default="" />
+  <!-- Load Spot -->
+  <xacro:load_spot
+    arm="$(arg arm)"
+    feet="$(arg feet)"
+    tf_prefix="$(arg tf_prefix)" />
 </robot>
