Commit message: Updated URDF to include mount points, and deps for install

File: spot_description/urdf/spot.urdf.xacro (robot description, xacro)
@@ -13,4 +13,16 @@
         </collision>
     </link>
+    <link name="front_rail"/>
+    <joint name="front_rail_joint" type="fixed">
+        <origin xyz="0.223 0 0.0805" rpy="0 0 0" />
+        <parent link="body" />
+        <child link="front_rail" />
+    </joint>
+    <link name="rear_rail"/>
+    <joint name="rear_rail_joint" type="fixed">
+        <origin xyz="-0.223 0 0.0805" rpy="0 0 0" />
+        <parent link="body" />
+        <child link="rear_rail" />
+    </joint>
     <link name="front_left_hip">
         <visual>

Commit message: Added base_link (rep-0105)

File: spot_description/urdf/spot.urdf.xacro (robot description, xacro)
@@ -13,4 +13,10 @@
         </collision>
     </link>
+    <link name="base_link"/>
+    <joint name="base_link_joint" type="fixed">
+        <origin xyz="0 0 0" rpy="0 0 0" />
+        <parent link="body" />
+        <child link="base_link" />
+    </joint>
     <link name="front_rail"/>
     <joint name="front_rail_joint" type="fixed">

Commit message: add correct joint for front rail, should be directly between first screws. Rear rail is based on that

File: spot_description/urdf/spot.urdf.xacro (robot description, xacro)
@@ -25,4 +25,10 @@
         <child link="front_rail" />
     </joint>
+    <link name="real_front_rail"/>
+    <joint name="real_front_rail_joint" type="fixed">
+        <origin xyz="0.2075 0 0.0805" rpy="0 0 0" />
+        <parent link="body" />
+        <child link="real_front_rail" />
+    </joint>
     <link name="rear_rail"/>
     <joint name="rear_rail_joint" type="fixed">
@@ -30,4 +36,10 @@
         <parent link="body" />
         <child link="rear_rail" />
+    </joint>
+    <link name="real_rear_rail"/>
+    <joint name="real_rear_rail_joint" type="fixed">
+        <origin xyz="-0.415 0 0" rpy="0 0 0" />
+        <parent link="real_front_rail" />
+        <child link="real_rear_rail" />
     </joint>
     <link name="front_left_hip">

Commit message: Add spot_champ_config and update URDF macros for CHAMP/Gazebo

File: spot_description/urdf/spot.urdf.xacro (robot description, xacro)
@@ -1,13 +1,10 @@
 <?xml version="1.0" ?>
-<robot name="spot" xmlns:xacro="http://www.ros.org/wiki/xacro">
+<robot name="spot"
+  xmlns:xacro="http://www.ros.org/wiki/xacro">
   <xacro:include filename="$(find spot_description)/urdf/spot_macro.xacro" />
   <!-- Parameters -->
   <xacro:arg name="arm" default="false" />
-  <xacro:arg name="feet" default="false" />
   <xacro:arg name="tf_prefix" default="" />
   <!-- Load Spot -->
-  <xacro:load_spot
-    arm="$(arg arm)"
-    feet="$(arg feet)"
-    tf_prefix="$(arg tf_prefix)" />
+  <xacro:load_spot arm="$(arg arm)" tf_prefix="$(arg tf_prefix)" />
 </robot>

File: spot_description/urdf/spot_macro.xacro (robot description, xacro)
@@ -1,7 +1,7 @@
 <?xml version="1.0"?>
-<robot name="spot" xmlns:xacro="http://www.ros.org/wiki/xacro">
-    <xacro:macro name="load_spot" params="
-    arm:=false
-    feet:=false
+<robot name="spot"
+    xmlns:xacro="http://www.ros.org/wiki/xacro">
+    <xacro:include filename="$(find spot_description)/urdf/constants.urdf.xacro" />
+    <xacro:macro name="load_spot" params=" arm:=false gazebo:=false
     tf_prefix">
         <link name="${tf_prefix}body">
@@ -13,16 +13,17 @@
             <collision>
                 <geometry>
-                    <mesh
-                        filename="package://spot_description/meshes/base/collision/body_collision.obj" />
+                    <mesh filename="package://spot_description/meshes/base/collision/body_collision.obj" />
                 </geometry>
             </collision>
+            <inertial>
+                <mass value="${base_mass}"/>
+                <inertia ixx="${(1/12) * base_mass * (base_width * base_width + base_height * base_height)}" ixy="0.0" ixz="0.0" iyy="${(1/12) * base_mass * (base_length * base_length + base_height * base_height)}" iyz="0.0" izz="${(1/12) * base_mass * (base_length * base_length + base_width * base_width)}" />
+            </inertial>
         </link>
         <link name="${tf_prefix}base_link">
             <inertial>
-                <origin rpy="0.0 0.0 0.0"
-                    xyz="0.006394396536052227 -9.812158532440662e-05 0.0009113792330026627" />
+                <origin rpy="0.0 0.0 0.0" xyz="0.006394396536052227 -9.812158532440662e-05 0.0009113792330026627" />
                 <mass value="32.86" />
-                <inertia ixx="0.13143999874591827" ixy="0.0" ixz="0.0" iyy="0.13143999874591827"
-                    iyz="0.0" izz="0.13143999874591827" />
+                <inertia ixx="0.13143999874591827" ixy="0.0" ixz="0.0" iyy="0.13143999874591827" iyz="0.0" izz="0.13143999874591827" />
             </inertial>
         </link>
@@ -56,348 +57,10 @@
             <child link="${tf_prefix}rear_rail" />
         </joint>
-        <link name="${tf_prefix}front_left_hip">
-            <visual>
-                <geometry>
-                    <mesh
-                        filename="package://spot_description/meshes/base/visual/front_left_hip.obj" />
-                </geometry>
-            </visual>
-            <inertial>
-                <origin rpy="-0.716521349312305 0.02956473059648479 0.03655230014702582"
-                    xyz="-0.005374345928430557 0.012841847725212574 9.875232353806496e-05" />
-                <mass value="1.68" />
-                <inertia ixx="0.0021147398873455382" ixy="0.0" ixz="0.0" iyy="0.0018129577956607131"
-                    iyz="0.0" izz="0.002265435737304666" />
-            </inertial>
-        </link>
-        <joint name="${tf_prefix}front_left_hip_x" type="revolute">
-            <origin xyz="0.29785 0.05500 0.00000" rpy="0 0 0" />
-            <axis xyz="1 0 0" />
-            <parent link="${tf_prefix}body" />
-            <child link="${tf_prefix}front_left_hip" />
-            <limit effort="45" velocity="17.647" lower="-0.78539816339744827899"
-                upper="0.78539816339744827899" />
-        </joint>
-        <link name="${tf_prefix}front_left_upper_leg">
-            <visual>
-                <geometry>
-                    <mesh
-                        filename="package://spot_description/meshes/base/visual/front_left_upper_leg.obj" />
-                </geometry>
-            </visual>
-            <collision>
-                <geometry>
-                    <mesh
-                        filename="package://spot_description/meshes/base/collision/left_upper_leg_collision.obj" />
-                </geometry>
-            </collision>
-            <inertial>
-                <origin rpy="-0.26437828203369795 -0.04853174570753804 0.024046963096353124"
-                    xyz="0.005142373498529196 -0.0024323679972440004 -0.12100915610790253" />
-                <mass value="2.34" />
-                <inertia ixx="0.02755964961185679" ixy="0.0" ixz="0.0" iyy="0.027354914287651046"
-                    iyz="0.0" izz="0.002848145546743553" />
-            </inertial>
-        </link>
-        <joint name="${tf_prefix}front_left_hip_y" type="revolute">
-            <origin xyz="0.0 0.110945 0.0" rpy="0 0 0" />
-            <axis xyz="0 1 0" />
-            <parent link="${tf_prefix}front_left_hip" />
-            <child link="${tf_prefix}front_left_upper_leg" />
-            <limit effort="45" velocity="17.647" lower="-0.89884456477707963539"
-                upper="2.2951079663725435509" />
-        </joint>
-        <link name="${tf_prefix}front_left_lower_leg">
-            <visual>
-                <geometry>
-                    <mesh
-                        filename="package://spot_description/meshes/base/visual/front_left_lower_leg.obj" />
-                </geometry>
-            </visual>
-            <collision>
-                <geometry>
-                    <mesh
-                        filename="package://spot_description/meshes/base/collision/left_lower_leg_collision.obj" />
-                </geometry>
-            </collision>
-            <collision>
-                <origin xyz="0.0 0.0 -0.3365" rpy="0 0 0" />
-                <geometry>
-                    <sphere radius="0.036"/>
-                </geometry>
-            </collision>
-            <inertial>
-                <origin rpy="-0.007266925694167092 -0.009591807116834161 0.00035255970529224356"
-                    xyz="0.00225794012658298 4.607596201822162e-05 -0.1800822913646698" />
-                <mass value="0.35" />
-                <inertia ixx="0.003999022654901177" ixy="0.0" ixz="0.0" iyy="0.0040503157598010785"
-                    iyz="0.0" izz="0.0001493402097647426" />
-            </inertial>
-        </link>
-        <joint name="${tf_prefix}front_left_knee" type="revolute">
-            <origin xyz="0.025 0.000 -0.3205" rpy="0 0 0" />
-            <axis xyz="0 1 0" />
-            <parent link="${tf_prefix}front_left_upper_leg" />
-            <child link="${tf_prefix}front_left_lower_leg" />
-            <limit effort="115" velocity="12.0" lower="-2.7929" upper="-0.254801" />
-        </joint>
-        <link name="${tf_prefix}front_right_hip">
-            <visual>
-                <geometry>
-                    <mesh
-                        filename="package://spot_description/meshes/base/visual/front_right_hip.obj" />
-                </geometry>
-            </visual>
-            <inertial>
-                <origin rpy="0.7165213493123055 -0.02956473059648479 0.03655230014702582"
-                    xyz="-0.005374345928430557 -0.012841847725212574 -9.875232353806496e-05" />
-                <mass value="1.68" />
-                <inertia ixx="0.0021147398873455382" ixy="0.0" ixz="0.0" iyy="0.0018129577956607131"
-                    iyz="0.0" izz="0.002265435737304666" />
-            </inertial>
-        </link>
-        <joint name="${tf_prefix}front_right_hip_x" type="revolute">
-            <origin xyz="0.29785 -0.05500 0.00000" rpy="0 0 0" />
-            <axis xyz="1 0 0" />
-            <parent link="${tf_prefix}body" />
-            <child link="${tf_prefix}front_right_hip" />
-            <limit effort="45" velocity="17.647" lower="-0.78539816339744827899"
-                upper="0.78539816339744827899" />
-        </joint>
-        <link name="${tf_prefix}front_right_upper_leg">
-            <visual>
-                <geometry>
-                    <mesh
-                        filename="package://spot_description/meshes/base/visual/front_right_upper_leg.obj" />
-                </geometry>
-            </visual>
-            <collision>
-                <geometry>
-                    <mesh
-                        filename="package://spot_description/meshes/base/collision/right_upper_leg_collision.obj" />
-                </geometry>
-            </collision>
-            <inertial>
-                <origin rpy="0.2643905306958363 -0.04853174688302708 -0.024046943559834943"
-                    xyz="0.005142373498529196 0.0024323677644133568 -0.12100915610790253" />
-                <mass value="2.34" />
-                <inertia ixx="0.02755964678927691" ixy="0.0" ixz="0.0" iyy="0.02735491706466737"
-                    iyz="0.0" izz="0.0028481453594764797" />
-            </inertial>
-        </link>
-        <joint name="${tf_prefix}front_right_hip_y" type="revolute">
-            <origin xyz="0.0 -0.110945 0.0" rpy="0 0 0" />
-            <axis xyz="0 1 0" />
-            <parent link="${tf_prefix}front_right_hip" />
-            <child link="${tf_prefix}front_right_upper_leg" />
-            <limit effort="45" velocity="17.647" lower="-0.89884456477707963539"
-                upper="2.2951079663725435509" />
-        </joint>
-        <link name="${tf_prefix}front_right_lower_leg">
-            <visual>
-                <geometry>
-                    <mesh
-                        filename="package://spot_description/meshes/base/visual/front_right_lower_leg.obj" />
-                </geometry>
-            </visual>
-            <collision>
-                <geometry>
-                    <mesh
-                        filename="package://spot_description/meshes/base/collision/right_lower_leg_collision.obj" />
-                </geometry>
-            </collision>
-            <collision>
-                <origin xyz="0.0 0.0 -0.3365" rpy="0 0 0" />
-                <geometry>
-                    <sphere radius="0.036"/>
-                </geometry>
-            </collision>
-            <inertial>
-                <origin rpy="-0.007266925694167092 -0.009591807116834161 0.00035255970529224356"
-                    xyz="0.00225794012658298 4.607596201822162e-05 -0.1800822913646698" />
-                <mass value="0.35" />
-                <inertia ixx="0.003999022654901177" ixy="0.0" ixz="0.0" iyy="0.0040503157598010785"
-                    iyz="0.0" izz="0.0001493402097647426" />
-            </inertial>
-        </link>
-        <joint name="${tf_prefix}front_right_knee" type="revolute">
-            <origin xyz="0.025 0.000 -0.3205" rpy="0 0 0" />
-            <axis xyz="0 1 0" />
-            <parent link="${tf_prefix}front_right_upper_leg" />
-            <child link="${tf_prefix}front_right_lower_leg" />
-            <limit effort="115" velocity="12.0" lower="-2.7929" upper="-0.247563" />
-        </joint>
-        <link name="${tf_prefix}rear_left_hip">
-            <visual>
-                <geometry>
-                    <mesh
-                        filename="package://spot_description/meshes/base/visual/rear_left_hip.obj" />
-                </geometry>
-            </visual>
-            <inertial>
-                <origin rpy="0.7165213493123055 -0.02956473059648479 0.03655230014702582"
-                    xyz="-0.005374345928430557 -0.012841847725212574 -9.875232353806496e-05" />
-                <mass value="1.68" />
-                <inertia ixx="0.0021147398873455382" ixy="0.0" ixz="0.0" iyy="0.0018129577956607131"
-                    iyz="0.0" izz="0.002265435737304666" />
-            </inertial>
-        </link>
-        <joint name="${tf_prefix}rear_left_hip_x" type="revolute">
-            <origin xyz="-0.29785 0.05500 0.00000" rpy="0 0 0" />
-            <axis xyz="1 0 0" />
-            <parent link="${tf_prefix}body" />
-            <child link="${tf_prefix}rear_left_hip" />
-            <limit effort="45" velocity="17.647" lower="-0.78539816339744827899"
-                upper="0.78539816339744827899" />
-        </joint>
-        <link name="${tf_prefix}rear_left_upper_leg">
-            <visual>
-                <geometry>
-                    <mesh
-                        filename="package://spot_description/meshes/base/visual/rear_left_upper_leg.obj" />
-                </geometry>
-            </visual>
-            <collision>
-                <geometry>
-                    <mesh
-                        filename="package://spot_description/meshes/base/collision/left_upper_leg_collision.obj" />
-                </geometry>
-            </collision>
-            <inertial>
-                <origin rpy="-0.26437828203369795 -0.04853174570753804 0.024046963096353124"
-                    xyz="0.005142373498529196 -0.0024323679972440004 -0.12100915610790253" />
-                <mass value="2.34" />
-                <inertia ixx="0.02755964961185679" ixy="0.0" ixz="0.0" iyy="0.027354914287651046"
-                    iyz="0.0" izz="0.002848145546743553" />
-            </inertial>
-        </link>
-        <joint name="${tf_prefix}rear_left_hip_y" type="revolute">
-            <origin xyz="0.0 0.110945 0.0" rpy="0 0 0" />
-            <axis xyz="0 1 0" />
-            <parent link="${tf_prefix}rear_left_hip" />
-            <child link="${tf_prefix}rear_left_upper_leg" />
-            <limit effort="45" velocity="17.647" lower="-0.89884456477707963539"
-                upper="2.2951079663725435509" />
-        </joint>
-        <link name="${tf_prefix}rear_left_lower_leg">
-            <visual>
-                <geometry>
-                    <mesh
-                        filename="package://spot_description/meshes/base/visual/rear_left_lower_leg.obj" />
-                </geometry>
-            </visual>
-            <collision>
-                <geometry>
-                    <mesh
-                        filename="package://spot_description/meshes/base/collision/left_lower_leg_collision.obj" />
-                </geometry>
-            </collision>
-            <collision>
-                <origin xyz="0.0 0.0 -0.3365" rpy="0 0 0" />
-                <geometry>
-                    <sphere radius="0.036"/>
-                </geometry>
-            </collision>
-            <inertial>
-                <origin rpy="-0.007266925694167092 -0.009591807116834161 0.00035255970529224356"
-                    xyz="0.00225794012658298 4.607596201822162e-05 -0.1800822913646698" />
-                <mass value="0.35" />
-                <inertia ixx="0.003999022654901177" ixy="0.0" ixz="0.0" iyy="0.0040503157598010785"
-                    iyz="0.0" izz="0.0001493402097647426" />
-            </inertial>
-        </link>
-        <joint name="${tf_prefix}rear_left_knee" type="revolute">
-            <origin xyz="0.025 0.000 -0.3205" rpy="0 0 0" />
-            <axis xyz="0 1 0" />
-            <parent link="${tf_prefix}rear_left_upper_leg" />
-            <child link="${tf_prefix}rear_left_lower_leg" />
-            <limit effort="115" velocity="12.0" lower="-2.7929" upper="-0.267153" />
-        </joint>
-        <link name="${tf_prefix}rear_right_hip">
-            <visual>
-                <geometry>
-                    <mesh
-                        filename="package://spot_description/meshes/base/visual/rear_right_hip.obj" />
-                </geometry>
-            </visual>
-            <inertial>
-                <origin rpy="0.7165213493123055 -0.02956473059648479 0.03655230014702582"
-                    xyz="-0.005374345928430557 -0.012841847725212574 -9.875232353806496e-05" />
-                <mass value="1.68" />
-                <inertia ixx="0.0021147398873455382" ixy="0.0" ixz="0.0" iyy="0.0018129577956607131"
-                    iyz="0.0" izz="0.002265435737304666" />
-            </inertial>
-        </link>
-        <joint name="${tf_prefix}rear_right_hip_x" type="revolute">
-            <origin xyz="-0.29785 -0.05500 0.00000" rpy="0 0 0" />
-            <axis xyz="1 0 0" />
-            <parent link="${tf_prefix}body" />
-            <child link="${tf_prefix}rear_right_hip" />
-            <limit effort="45" velocity="17.647" lower="-0.78539816339744827899"
-                upper="0.78539816339744827899" />
-        </joint>
-        <link name="${tf_prefix}rear_right_upper_leg">
-            <visual>
-                <geometry>
-                    <mesh
-                        filename="package://spot_description/meshes/base/visual/rear_right_upper_leg.obj" />
-                </geometry>
-            </visual>
-            <collision>
-                <geometry>
-                    <mesh
-                        filename="package://spot_description/meshes/base/collision/right_upper_leg_collision.obj" />
-                </geometry>
-            </collision>
-            <inertial>
-                <origin rpy="0.2643905306958363 -0.04853174688302708 -0.024046943559834943"
-                    xyz="0.005142373498529196 0.0024323677644133568 -0.12100915610790253" />
-                <mass value="2.34" />
-                <inertia ixx="0.02755964678927691" ixy="0.0" ixz="0.0" iyy="0.02735491706466737"
-                    iyz="0.0" izz="0.0028481453594764797" />
-            </inertial>
-        </link>
-        <joint name="${tf_prefix}rear_right_hip_y" type="revolute">
-            <origin xyz="0.0 -0.110945 0.0" rpy="0 0 0" />
-            <axis xyz="0 1 0" />
-            <parent link="${tf_prefix}rear_right_hip" />
-            <child link="${tf_prefix}rear_right_upper_leg" />
-            <limit effort="45" velocity="17.647" lower="-0.89884456477707963539"
-                upper="2.2951079663725435509" />
-        </joint>
-        <link name="${tf_prefix}rear_right_lower_leg">
-            <visual>
-                <geometry>
-                    <mesh
-                        filename="package://spot_description/meshes/base/visual/rear_right_lower_leg.obj" />
-                </geometry>
-            </visual>
-            <collision>
-                <geometry>
-                    <mesh
-                        filename="package://spot_description/meshes/base/collision/right_lower_leg_collision.obj" />
-                </geometry>
-            </collision>
-            <collision>
-                <origin xyz="0.0 0.0 -0.3365" rpy="0 0 0" />
-                <geometry>
-                    <sphere radius="0.036"/>
-                </geometry>
-            </collision>
-            <inertial>
-                <origin rpy="-0.007266925694167092 -0.009591807116834161 0.00035255970529224356"
-                    xyz="0.00225794012658298 4.607596201822162e-05 -0.1800822913646698" />
-                <mass value="0.35" />
-                <inertia ixx="0.003999022654901177" ixy="0.0" ixz="0.0" iyy="0.0040503157598010785"
-                    iyz="0.0" izz="0.0001493402097647426" />
-            </inertial>
-        </link>
-        <joint name="${tf_prefix}rear_right_knee" type="revolute">
-            <origin xyz="0.025 0.000 -0.3205" rpy="0 0 0" />
-            <axis xyz="0 1 0" />
-            <parent link="${tf_prefix}rear_right_upper_leg" />
-            <child link="${tf_prefix}rear_right_lower_leg" />
-            <limit effort="115" velocity="12.0" lower="-2.7929" upper="-0.257725" />
-        </joint>
+        <!-- Macros for Spot's legs. -->
+        <xacro:include filename="$(find spot_description)/urdf/spot_leg.urdf.xacro" />
+        <xacro:spot_leg leg_name="front_left"/>
+        <xacro:spot_leg leg_name="front_right"/>
+        <xacro:spot_leg leg_name="rear_left"/>
+        <xacro:spot_leg leg_name="rear_right"/>
         <!-- Standard accessories. -->
         <xacro:include filename="$(find spot_description)/urdf/accessories.urdf.xacro" />
@@ -409,8 +72,23 @@
             <xacro:load_arm tf_prefix="${tf_prefix}" />
         </xacro:if>
-        <!-- Include links at feet if necessary -->
-        <xacro:if value="${feet}">
-            <xacro:include filename="$(find spot_description)/urdf/spot_feet_macro.urdf" />
-            <xacro:load_feet tf_prefix="${tf_prefix}" />
+        <!-- Include Gazebo control if necessary -->
+        <xacro:if value="${gazebo}">
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